Commit message: file: legged_example/humanoid/humanoid_description state: error, need create xacro

File: src/legged_examples/humanoid/humanoid_description/urdf/humanoid.urdf (robot description, URDF)
Before this commit: robot humanoid, 17 links, 16 joints
Links:
- link L_Foot: geometry collision sphere radius=0.0; collision sphere radius=0.0
- link L_ForeArm: geometry visual mesh filename=package://humanoid_description/meshes_zidong_obj/L_ForeArm2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 scale=1 1 1
- link L_HipRx: geometry visual mesh filename=package://humanoid_description/meshes_zidong_obj/L_HipRx.dae scale=1 1 1
- link L_HipRz: geometry visual mesh filename=package://humanoid_description/meshes_zidong_obj/R_HipRz.dae scale=1 1 1
- link L_Shank: geometry visual mesh filename=package://humanoid_description/meshes_zidong_obj/L_LowerLeg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 scale=1 1 1
- link L_ShoulderRx: geometry visual mesh filename=package://humanoid_description/meshes_zidong_obj/R_Shoulder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 scale=1 1 1
- link L_Thigh: geometry visual mesh filename=package://humanoid_description/meshes_zidong_obj/L_Thigh.dae scale=1 1 1
- link L_UpperArm: geometry visual mesh filename=package://humanoid_description/meshes_zidong_obj/L_UpperArm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 scale=1 1 1
- link R_Foot: geometry collision sphere radius=0.0; collision sphere radius=0.0
- link R_ForeArm: geometry visual mesh filename=package://humanoid_description/meshes_zidong_obj/L_ForeArm2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 scale=1 1 1
- link R_HipRx: geometry visual mesh filename=package://humanoid_description/meshes_zidong_obj/R_HipRx.dae scale=1 1 1
- link R_HipRz: geometry visual mesh filename=package://humanoid_description/meshes_zidong_obj/R_HipRz.dae scale=1 1 1
- link R_Shank: geometry visual mesh filename=package://humanoid_description/meshes_zidong_obj/R_LowerLeg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 scale=1 1 1
- link R_ShoulderRx: geometry visual mesh filename=package://humanoid_description/meshes_zidong_obj/R_Shoulder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 scale=1 1 1
- link R_Thigh: geometry visual mesh filename=package://humanoid_description/meshes_zidong_obj/R_Thigh.dae scale=1 1 1
- link R_UpperArm: geometry visual mesh filename=package://humanoid_description/meshes_zidong_obj/R_UpperArm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 scale=1 1 1
- link torso: geometry visual mesh filename=package://humanoid_description/meshes_zidong_obj/Body.dae scale=1 1 1
