Commit message: correct pinocchio_interface.np=6

File: src/ocs2_robotic_assets/resources/anymal_c/urdf/anymal.urdf (robot description, URDF)
Before this commit: robot anymal, 78 links, 77 joints
Links:
- removed link LF_FOOT
- removed link LF_HAA
- removed link LF_HFE
- removed link LF_HIP
- removed link LF_KFE
- removed link LF_SHANK
- removed link LF_THIGH
- removed link LF_hip_fixed
- removed link LF_shank_fixed
- removed link LF_thigh_fixed
- removed link LH_FOOT
- removed link LH_HAA
- removed link LH_HFE
- removed link LH_HIP
- removed link LH_KFE
- removed link LH_SHANK
- removed link LH_THIGH
- removed link LH_hip_fixed
- removed link LH_shank_fixed
- removed link LH_thigh_fixed
- removed link RF_FOOT
- removed link RF_HAA
- removed link RF_HFE
- removed link RF_HIP
- removed link RF_KFE
- removed link RF_SHANK
- removed link RF_THIGH
- removed link RF_hip_fixed
- removed link RF_shank_fixed
- removed link RF_thigh_fixed
- removed link RH_FOOT
- removed link RH_HAA
- removed link RH_HFE
- removed link RH_HIP
- removed link RH_KFE
- removed link RH_SHANK
- removed link RH_THIGH
- removed link RH_hip_fixed
- removed link RH_shank_fixed
- removed link RH_thigh_fixed
- removed link base
- removed link base_inertia
- removed link battery
- removed link bottom_shell
- removed link depth_camera_front_camera
- removed link depth_camera_front_camera_parent
- removed link depth_camera_front_color_frame
- removed link depth_camera_front_color_optical_frame
- removed link depth_camera_front_depth_optical_frame
- removed link depth_camera_left_camera
- removed link depth_camera_left_camera_parent
- removed link depth_camera_left_color_frame
- removed link depth_camera_left_color_optical_frame
- removed link depth_camera_left_depth_optical_frame
- removed link depth_camera_rear_camera
- removed link depth_camera_rear_camera_parent
- removed link depth_camera_rear_color_frame
- removed link depth_camera_rear_color_optical_frame
- removed link depth_camera_rear_depth_optical_frame
- removed link depth_camera_right_camera
- removed link depth_camera_right_camera_parent
- removed link depth_camera_right_color_frame
- removed link depth_camera_right_color_optical_frame
- removed link depth_camera_right_depth_optical_frame
- removed link docking_hatch_cover
- removed link face_front
- removed link face_rear
- removed link handle
- removed link hatch
- removed link imu_link
- removed link lidar
- removed link lidar_cage
- removed link remote
- removed link top_shell
- removed link wide_angle_camera_front_camera
- removed link wide_angle_camera_front_camera_parent
- removed link wide_angle_camera_rear_camera
- removed link wide_angle_camera_rear_camera_parent
- added link L_Foot, mass 0.30; collision sphere radius=0.0; collision sphere radius=0.0
- added link L_ForeArm, mass 0.1; visual mesh filename=package://ocs2_robotic_assets/resources/anymal_c/meshes_zid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 scale=1 1 1
- added link L_HipRx, mass 0.30; visual mesh filename=package://ocs2_robotic_assets/resources/anymal_c/meshes_zid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 scale=1 1 1
- added link L_HipRz, mass 0.30; visual mesh filename=package://ocs2_robotic_assets/resources/anymal_c/meshes_zid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 scale=1 1 1
- added link L_Shank, mass 0.70; visual mesh filename=package://ocs2_robotic_assets/resources/anymal_c/meshes_zid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 scale=1 1 1
- added link L_ShoulderRx, mass 0.30; visual mesh filename=package://ocs2_robotic_assets/resources/anymal_c/meshes_zid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 scale=1 1 1
- added link L_Thigh, mass 1.0; visual mesh filename=package://ocs2_robotic_assets/resources/anymal_c/meshes_zid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 scale=1 1 1
- added link L_UpperArm, mass 0.37; visual mesh filename=package://ocs2_robotic_assets/resources/anymal_c/meshes_zid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 scale=1 1 1
- added link R_Foot, mass 0.30; collision sphere radius=0.0; collision sphere radius=0.0
- added link R_ForeArm, mass 0.1; visual mesh filename=package://ocs2_robotic_assets/resources/anymal_c/meshes_zid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 scale=1 1 1
- added link R_HipRx, mass 0.30; visual mesh filename=package://ocs2_robotic_assets/resources/anymal_c/meshes_zid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 scale=1 1 1
- added link R_HipRz, mass 0.30; visual mesh filename=package://ocs2_robotic_assets/resources/anymal_c/meshes_zid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 scale=1 1 1
- added link R_Shank, mass 0.70; visual mesh filename=package://ocs2_robotic_assets/resources/anymal_c/meshes_zid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 scale=1 1 1
- added link R_ShoulderRx, mass 0.30; visual mesh filename=package://ocs2_robotic_assets/resources/anymal_c/meshes_zid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 scale=1 1 1
- added link R_Thigh, mass 1.0; visual mesh filename=package://ocs2_robotic_assets/resources/anymal_c/meshes_zid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 scale=1 1 1
- added link R_UpperArm, mass 0.37; visual mesh filename=package://ocs2_robotic_assets/resources/anymal_c/meshes_zid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 scale=1 1 1
- added link torso, mass 6.5; visual mesh filename=package://ocs2_robotic_assets/resources/anymal_c/meshes_zid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 scale=1 1 1
Joints:
- removed joint LF_HAA
- removed joint LF_HFE
- removed joint LF_HIP_LF_hip_fixed
- removed joint LF_KFE
- removed joint LF_THIGH_LF_thigh_fixed
- removed joint LF_hip_fixed_LF_HFE
- removed joint LF_shank_LF_shank_fixed
- removed joint LF_shank_fixed_LF_FOOT
- removed joint LF_thigh_fixed_LF_KFE
- removed joint LH_HAA
- removed joint LH_HFE
- removed joint LH_HIP_LH_hip_fixed
- removed joint LH_KFE
- removed joint LH_THIGH_LH_thigh_fixed
- removed joint LH_hip_fixed_LH_HFE
- removed joint LH_shank_LH_shank_fixed
- removed joint LH_shank_fixed_LH_FOOT
- removed joint LH_thigh_fixed_LH_KFE
- removed joint RF_HAA
- removed joint RF_HFE
- removed joint RF_HIP_RF_hip_fixed
- removed joint RF_KFE
- removed joint RF_THIGH_RF_thigh_fixed
- removed joint RF_hip_fixed_RF_HFE
- removed joint RF_shank_RF_shank_fixed
- removed joint RF_shank_fixed_RF_FOOT
- removed joint RF_thigh_fixed_RF_KFE
- removed joint RH_HAA
- removed joint RH_HFE
- removed joint RH_HIP_RH_hip_fixed
- removed joint RH_KFE
- removed joint RH_THIGH_RH_thigh_fixed
- removed joint RH_hip_fixed_RH_HFE
- removed joint RH_shank_RH_shank_fixed
- removed joint RH_shank_fixed_RH_FOOT
- removed joint RH_thigh_fixed_RH_KFE
- removed joint base_LF_HAA
- removed joint base_LH_HAA
- removed joint base_RF_HAA
- removed joint base_RH_HAA
- removed joint base_battery
- removed joint base_bottom_shell
- removed joint base_face_front
- removed joint base_face_rear
- removed joint base_handle
- removed joint base_hatch
- removed joint base_remote
- removed joint base_to_base_inertia
- removed joint base_to_depth_camera_left_camera
- removed joint base_to_depth_camera_right_camera
- removed joint base_to_docking_hatch_cover
- removed joint base_to_lidar_cage
- removed joint base_top_shell
- removed joint depth_camera_front_camera_parent_to_color_frame
- removed joint depth_camera_front_camera_parent_to_depth_optical_frame
- removed joint depth_camera_front_camera_to_camera_parent
- removed joint depth_camera_front_color_frame_to_color_optical_frame
- removed joint depth_camera_left_camera_parent_to_color_frame
- removed joint depth_camera_left_camera_parent_to_depth_optical_frame
- removed joint depth_camera_left_camera_to_camera_parent
- removed joint depth_camera_left_color_frame_to_color_optical_frame
- removed joint depth_camera_rear_camera_parent_to_color_frame
- removed joint depth_camera_rear_camera_parent_to_depth_optical_frame
- removed joint depth_camera_rear_camera_to_camera_parent
- removed joint depth_camera_rear_color_frame_to_color_optical_frame
- removed joint depth_camera_right_camera_parent_to_color_frame
- removed joint depth_camera_right_camera_parent_to_depth_optical_frame
- removed joint depth_camera_right_camera_to_camera_parent
- removed joint depth_camera_right_color_frame_to_color_optical_frame
- removed joint face_front_to_depth_camera_front_camera
- removed joint face_front_to_wide_angle_camera_front_camera
- removed joint face_rear_to_depth_camera_rear_camera
- removed joint face_rear_to_wide_angle_camera_rear_camera
- removed joint imu_joint
- removed joint lidar_cage_to_lidar
- removed joint wide_angle_camera_front_camera_to_camera_parent
- removed joint wide_angle_camera_rear_camera_to_camera_parent
- added joint L_Ankle: type revolute, parent L_Shank, child L_Foot, origin xyz=0.0 0.0 -0.247 rpy=0 0 0, axis 0 1 0, limit lower=-3 upper=3 effort=33.6 velocity=55
- added joint L_HipRx_to_L_Thigh: type revolute, parent L_HipRx, child L_Thigh, origin xyz=0.065 0.0 0.0 rpy=0 0 0, axis 0 1 0, limit lower=-3 upper=3 effort=33.6 velocity=55
- added joint L_HipRz_to_L_HipRx: type revolute, parent L_HipRz, child L_HipRx, origin xyz=-0.041 0.0 -0.0885 rpy=0 0 0, axis 1 0 0, limit lower=-3 upper=3 effort=33.6 velocity=55
- added joint L_Knee: type revolute, parent L_Thigh, child L_Shank, origin xyz=0.0 -0.017875 -0.247 rpy=0 0 0, axis 0 1 0, limit lower=-3 upper=3 effort=33.6 velocity=55
- added joint L_ShoulderRx_to_L_UpperArm: type revolute, parent L_ShoulderRx, child L_UpperArm, origin xyz=0.0545 0.0 0.0 rpy=0 0 0, axis 0 1 0, limit lower=-3 upper=3 effort=33.6 velocity=55
- added joint L_UpperArm_to_L_ForeArm: type revolute, parent L_UpperArm, child L_ForeArm, origin xyz=0.0 0.068 -0.195 rpy=0 0 0, axis 0 1 0, limit lower=-3 upper=3 effort=33.6 velocity=55
- added joint R_Ankle: type revolute, parent R_Shank, child R_Foot, origin xyz=0.0 0.0 -0.247 rpy=0 0 0, axis 0 1 0, limit lower=-3 upper=3 effort=33.6 velocity=55
- added joint R_HipRx_to_R_Thigh: type revolute, parent R_HipRx, child R_Thigh, origin xyz=0.065 0.0 0.0 rpy=0 0 0, axis 0 1 0, limit lower=-3 upper=3 effort=33.6 velocity=55
- added joint R_HipRz_to_R_HipRx: type revolute, parent R_HipRz, child R_HipRx, origin xyz=-0.041 0.0 -0.0885 rpy=0 0 0, axis 1 0 0, limit lower=-3 upper=3 effort=33.6 velocity=55
- added joint R_Knee: type revolute, parent R_Thigh, child R_Shank, origin xyz=0.0 0.017875 -0.247 rpy=0 0 0, axis 0 1 0, limit lower=-3 upper=3 effort=33.6 velocity=55
- added joint R_ShoulderRx_to_R_UpperArm: type revolute, parent R_ShoulderRx, child R_UpperArm, origin xyz=0.0545 0.0 0.0 rpy=0 0 0, axis 0 1 0, limit lower=-3 upper=3 effort=33.6 velocity=55
- added joint R_UpperArm_to_R_ForeArm: type revolute, parent R_UpperArm, child R_ForeArm, origin xyz=0.0 -0.068 -0.195 rpy=0 0 0, axis 0 1 0, limit lower=-3 upper=3 effort=33.6 velocity=55
- added joint torso_to_L_HipRz: type revolute, parent torso, child L_HipRz, origin xyz=0.0 0.075 0.0 rpy=0 0 0, axis 0 0 1, limit lower=-3 upper=3 effort=33.6 velocity=55
- added joint torso_to_L_ShoulderRx: type revolute, parent torso, child L_ShoulderRx, origin xyz=-0.0215 0.1115 0.202 rpy=0 0 0, axis 1 0 0, limit lower=-3 upper=3 effort=33.6 velocity=55
- added joint torso_to_R_HipRz: type revolute, parent torso, child R_HipRz, origin xyz=0.0 -0.075 0.0 rpy=0 0 0, axis 0 0 1, limit lower=-3 upper=3 effort=33.6 velocity=55
- added joint torso_to_R_ShoulderRx: type revolute, parent torso, child R_ShoulderRx, origin xyz=-0.0215 -0.1115 0.202 rpy=0 0 0, axis 1 0 0, limit lower=-3 upper=3 effort=33.6 velocity=55

Commit message: getPositionComToContactPointInWorldFrame wrong

File: src/ocs2_robotic_assets/resources/anymal_c/urdf/anymal.urdf (robot description, URDF)
Before this commit: robot humanoid, 17 links, 16 joints
Links:
- removed link L_ForeArm
- removed link L_HipRx
- removed link L_HipRz
- removed link L_Shank
- removed link L_ShoulderRx
- removed link L_Thigh
- removed link L_UpperArm
- removed link R_ForeArm
- removed link R_HipRx
- removed link R_HipRz
- removed link R_Shank
- removed link R_ShoulderRx
- removed link R_Thigh
- removed link R_UpperArm
- removed link torso
- added link L_LForeArm, mass 0.1; visual mesh filename=package://legged_unitree_description/meshes/a1/L_ForeArm2.o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 scale=1 1 1; visual mesh filename=package://legged_unitree_description/meshes/a1/R_ShoulderRx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 scale=1 1 1
- added link L_LHipRx, mass 0.30; visual mesh filename=package://legged_unitree_description/meshes/a1/L_HipRx.obj scale=1 1 1
- added link L_LHipRz, mass 0.30; visual mesh filename=package://legged_unitree_description/meshes/a1/L_HipRz.obj scale=1 1 1
- added link L_LShank, mass 0.70; visual mesh filename=package://legged_unitree_description/meshes/a1/L_LowerLeg3_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 scale=1 1 1
- added link L_LShoulderRx, mass 0.30; visual mesh filename=package://legged_unitree_description/meshes/a1/L_ShoulderRx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 scale=1 1 1
- added link L_LThigh, mass 1.0; visual mesh filename=package://legged_unitree_description/meshes/a1/L_Thigh.obj scale=1 1 1
- added link L_LUpperArm, mass 0.37; visual mesh filename=package://legged_unitree_description/meshes/a1/L_UpperArm.o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 scale=1 1 1
- added link R_LForeArm, mass 0.1; visual mesh filename=package://legged_unitree_description/meshes/a1/R_ForeArm2.o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 scale=1 1 1; visual mesh filename=package://legged_unitree_description/meshes/a1/R_ShoulderRx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 scale=1 1 1
- added link R_LHipRx, mass 0.30; visual mesh filename=package://legged_unitree_description/meshes/a1/R_HipRx.obj scale=1 1 1
- added link R_LHipRz, mass 0.30; visual mesh filename=package://legged_unitree_description/meshes/a1/R_HipRz.obj scale=1 1 1
- added link R_LShank, mass 0.70; visual mesh filename=package://legged_unitree_description/meshes/a1/R_LowerLeg3_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 scale=1 1 1
- added link R_LShoulderRx, mass 0.30; visual mesh filename=package://legged_unitree_description/meshes/a1/L_ShoulderRx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 scale=1 1 1
- added link R_LThigh, mass 1.0; visual mesh filename=package://legged_unitree_description/meshes/a1/R_Thigh.obj scale=1 1 1
- added link R_LUpperArm, mass 0.37; visual mesh filename=package://legged_unitree_description/meshes/a1/R_UpperArm.o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 scale=1 1 1
- added link base, mass 6.5; collision box size=0.267 0.194 0.114; visual mesh filename=package://legged_unitree_description/meshes/a1/Body.obj scale=1 1 1
- added link unitree_imu, mass 0.01; visual box size=0.015 0.015 0.004
- link L_Foot: geometry collision sphere radius=0.0; collision sphere radius=0.0
- link R_Foot: geometry collision sphere radius=0.0; collision sphere radius=0.0
Joints:
- removed joint L_Ankle
- removed joint L_HipRx_to_L_Thigh
- removed joint L_HipRz_to_L_HipRx
- removed joint L_Knee
- removed joint L_ShoulderRx_to_L_UpperArm
- removed joint L_UpperArm_to_L_ForeArm
- removed joint R_Ankle
- removed joint R_HipRx_to_R_Thigh
- removed joint R_HipRz_to_R_HipRx
- removed joint R_Knee
- removed joint R_ShoulderRx_to_R_UpperArm
- removed joint R_UpperArm_to_R_ForeArm
- removed joint torso_to_L_HipRz
- removed joint torso_to_L_ShoulderRx
- removed joint torso_to_R_HipRz
- removed joint torso_to_R_ShoulderRx
- added joint L_JAnkle: type revolute, parent L_LShank, child L_Foot, origin xyz=0.0 0.0 -0.247 rpy=0 0 0, axis 0 1 0, limit lower=-3 upper=3 effort=33.5 velocity=33.5
- added joint L_JForeArm: type revolute, parent L_LUpperArm, child L_LForeArm, origin xyz=0.0 0.068 -0.195 rpy=0 0 0, axis 0 1 0, limit lower=-3 upper=3 effort=33.5 velocity=33.5
- added joint L_JHipRx: type revolute, parent L_LHipRz, child L_LHipRx, origin xyz=-0.041 0.0 -0.0885 rpy=0 0 0, axis 1 0 0, limit lower=-3 upper=3 effort=33.5 velocity=33.5
- added joint L_JHipRz: type revolute, parent base, child L_LHipRz, origin xyz=0 0.075 0 rpy=0 0 0, axis 0 0 1, limit lower=-3 upper=3 effort=33.5 velocity=21
- added joint L_JKnee: type revolute, parent L_LThigh, child L_LShank, origin xyz=0.0 -0.017875 -0.247 rpy=0 0 0, axis 0 1 0, limit lower=-3 upper=3 effort=33.5 velocity=33.5
- added joint L_JShoulderRx: type revolute, parent base, child L_LShoulderRx, origin xyz=-0.0215 0.1115 0.202 rpy=0 0 0, axis 1 0 0, limit lower=-3 upper=3 effort=33.5 velocity=21
- added joint L_JThigh: type revolute, parent L_LHipRx, child L_LThigh, origin xyz=0.065 0.0 0.0 rpy=0 0 0, axis 0 1 0, limit lower=-3 upper=3 effort=33.5 velocity=33.5
- added joint L_JUpperArm: type revolute, parent L_LShoulderRx, child L_LUpperArm, origin xyz=0.0545 0.0 0.0 rpy=0 0 0, axis 0 1 0, limit lower=-3 upper=3 effort=33.5 velocity=33.5
- added joint R_JAnkle: type revolute, parent R_LShank, child R_Foot, origin xyz=0.0 0.0 -0.247 rpy=0 0 0, axis 0 1 0, limit lower=-3 upper=3 effort=33.5 velocity=33.5
- added joint R_JForeArm: type revolute, parent R_LUpperArm, child R_LForeArm, origin xyz=0.0 -0.068 -0.195 rpy=0 0 0, axis 0 1 0, limit lower=-3 upper=3 effort=33.5 velocity=33.5
- added joint R_JHipRx: type revolute, parent R_LHipRz, child R_LHipRx, origin xyz=-0.041 0.0 -0.0885 rpy=0 0 0, axis 1 0 0, limit lower=-3 upper=3 effort=33.5 velocity=33.5
- added joint R_JHipRz: type revolute, parent base, child R_LHipRz, origin xyz=0 -0.075 0 rpy=0 0 0, axis 0 0 1, limit lower=-3 upper=3 effort=33.5 velocity=21
- added joint R_JKnee: type revolute, parent R_LThigh, child R_LShank, origin xyz=0.0 0.017875 -0.247 rpy=0 0 0, axis 0 1 0, limit lower=-3 upper=3 effort=33.5 velocity=33.5
- added joint R_JShoulderRx: type revolute, parent base, child R_LShoulderRx, origin xyz=-0.0215 -0.1115 0.202 rpy=0 0 0, axis 1 0 0, limit lower=-3 upper=3 effort=33.5 velocity=21
- added joint R_JThigh: type revolute, parent R_LHipRx, child R_LThigh, origin xyz=0.065 0.0 0.0 rpy=0 0 0, axis 0 1 0, limit lower=-3 upper=3 effort=33.5 velocity=33.5
- added joint R_JUpperArm: type revolute, parent R_LShoulderRx, child R_LUpperArm, origin xyz=0.0545 0.0 0.0 rpy=0 0 0, axis 0 1 0, limit lower=-3 upper=3 effort=33.5 velocity=33.5
- added joint unitree_imu_joint: type fixed, parent base, child unitree_imu, origin xyz=0. 0. 0. rpy=0. 0. 0.
