Commit message: robot.xacro --> edit from qua --> bipedal

File: src/legged_examples/legged_unitree/legged_unitree_description/urdf/common/arm.xacro (robot description, xacro)
@@ -31,5 +31,5 @@
         <joint name="${prefix}_JUpperArm" type="revolute">
             <origin rpy="0 0 0" xyz="0.0545 0.0 0.0"/>
-            <parent link="${prefix}__LShoulderRx"/>
+            <parent link="${prefix}_LShoulderRx"/>
             <child link="${prefix}_LUpperArm"/>
             <axis xyz="0 1 0"/>
@@ -40,5 +40,5 @@
         <link name="${prefix}_LUpperArm">
             <visual>
-                <origin rpy="0 1.57 -1.57" xyz="0. 0.07*mirror 0"/>
+                <origin rpy="0 1.57 -1.57" xyz="0. ${0.07*mirror} 0"/>
                 <geometry>
                     <mesh filename="package://legged_unitree_description/meshes/$(arg robot_type)/${prefix}_UpperArm.dae"
@@ -57,6 +57,6 @@
         </link>
         <joint name="${prefix}_JForeArm" type="revolute">
-            <origin rpy="0 0 0" xyz="0.0 0.068*mirror -0.195"/>
-            <parent link="${prefix}__LUpperArm"/>
+            <origin rpy="0 0 0" xyz="0.0 ${0.068*mirror} -0.195"/>
+            <parent link="${prefix}_LUpperArm"/>
             <child link="${prefix}_LForeArm"/>
             <axis xyz="0 1 0"/>

File: src/legged_examples/legged_unitree/legged_unitree_description/urdf/common/leg.xacro (robot description, xacro)
@@ -31,5 +31,5 @@
         <joint name="${prefix}_JHipRx" type="revolute">
             <origin rpy="0 0 0" xyz="-0.041 0.0 -0.0885"/>
-            <parent link="${prefix}__LHipRz"/>
+            <parent link="${prefix}_LHipRz"/>
             <child link="${prefix}_LHipRx"/>
             <axis xyz="1 0 0"/>
@@ -58,5 +58,5 @@
         <joint name="${prefix}_JThigh" type="revolute">
             <origin rpy="0 0 0" xyz="0.065 0.0 0.0"/>
-            <parent link="${prefix}__LHipRx"/>
+            <parent link="${prefix}_LHipRx"/>
             <child link="${prefix}_LThigh"/>
             <axis xyz="0 1 0"/>
@@ -84,6 +84,6 @@
         </link>
         <joint name="${prefix}_JKnee" type="revolute">
-            <origin rpy="0 0 0" xyz="0.0 -0.017875*mirror -0.247"/>
-            <parent link="${prefix}__LThigh"/>
+            <origin rpy="0 0 0" xyz="0.0 ${-0.017875*mirror} -0.247"/>
+            <parent link="${prefix}_LThigh"/>
             <child link="${prefix}_LShank"/>
             <axis xyz="0 1 0"/>
@@ -112,5 +112,5 @@
         <joint name="${prefix}_JAnkle" type="revolute">
             <origin rpy="0 0 0" xyz="0.0 0.0 -0.247"/>
-            <parent link="${prefix}__LShank"/>
+            <parent link="${prefix}_LShank"/>
             <child link="${prefix}_Foot"/>
             <axis xyz="0 1 0"/>

File: src/legged_examples/legged_unitree/legged_unitree_description/urdf/robot.xacro (robot description, xacro)
@@ -37,9 +37,9 @@
         <origin rpy="0 0 0" xyz="0 -0.075 0"/>
     </xacro:leg>
-    <xacro:arm prefix="L" mirror="1" mirror_dae="False" front_hind="1" front_hind_dae="True">
+    <xacro:arm prefix="L" mirror="1.0" mirror_dae="False" front_hind="1" front_hind_dae="True">
         <origin rpy="0 0 0" xyz="-0.0215 0.1115 0.202"/>
-    </xacro:leg>
-    <xacro:arm prefix="R" mirror="-1" mirror_dae="True" front_hind="1" front_hind_dae="True">
+    </xacro:arm>
+    <xacro:arm prefix="R" mirror="-1.0" mirror_dae="True" front_hind="1" front_hind_dae="True">
         <origin rpy="0 0 0" xyz="-0.0215 -0.1115 0.202"/>
-    </xacro:leg>
+    </xacro:arm>
 </robot>

Commit message: edit arm

File: src/legged_examples/legged_unitree/legged_unitree_description/urdf/common/arm.xacro (robot description, xacro)
@@ -13,5 +13,5 @@
         <link name="${prefix}_LShoulderRx">
             <visual>
-                <origin rpy="0 0 0.0" xyz="0.06 0.02 -0.055"/>
+                <origin rpy="0 0 0.0" xyz="0 0 0.0"/>
                 <geometry>
                     <mesh filename="package://legged_unitree_description/meshes/$(arg robot_type)/${prefix}_ShoulderRx.dae"
@@ -40,5 +40,10 @@
         <link name="${prefix}_LUpperArm">
             <visual>
-                <origin rpy="0 1.57 -1.57" xyz="0. ${0.07*mirror} 0"/>
+            <xacro:if value="${(mirror == True)}">
+                <origin rpy="0 1.57 -1.57" xyz="0. 0.07 0"/>
+            </xacro:if>
+            <xacro:if value="${(mirror == False)}">
+                <origin rpy="0 0 0.0" xyz="0 0 0.0"/>
+            </xacro:if>
                 <geometry>
                     <mesh filename="package://legged_unitree_description/meshes/$(arg robot_type)/${prefix}_UpperArm.dae"
@@ -67,5 +72,5 @@
         <link name="${prefix}_LForeArm">
             <visual>
-                <origin rpy="0 1.57 0" xyz="0. 0 0"/>
+                <origin rpy="0 0 0.0" xyz="0. 0 0"/>
                 <geometry>
                     <mesh filename="package://legged_unitree_description/meshes/$(arg robot_type)/${prefix}_ForeArm2.dae"

Commit message: upper model correct

File: src/legged_examples/legged_unitree/legged_unitree_description/urdf/common/arm.xacro (robot description, xacro)
@@ -13,5 +13,5 @@
         <link name="${prefix}_LShoulderRx">
             <visual>
-                <origin rpy="0 0 0.0" xyz="0 0 0.0"/>
+                <origin rpy="0 0 0.0" xyz="0 0.0 0.0"/>
                 <geometry>
                     <mesh filename="package://legged_unitree_description/meshes/$(arg robot_type)/${prefix}_ShoulderRx.dae"
@@ -41,5 +41,5 @@
             <visual>
             <xacro:if value="${(mirror == True)}">
-                <origin rpy="0 1.57 -1.57" xyz="0. 0.07 0"/>
+                <origin rpy="0 0 -3.14" xyz="0. 0.0 0"/>
             </xacro:if>
             <xacro:if value="${(mirror == False)}">

Commit message: upper correct; dae-->obj

File: src/legged_examples/legged_unitree/legged_unitree_description/urdf/common/arm.xacro (robot description, xacro)
@@ -13,10 +13,15 @@
         <link name="${prefix}_LShoulderRx">
             <visual>
-                <origin rpy="0 0 0.0" xyz="0 0.0 0.0"/>
+                <xacro:if value="${(mirror == True)}">
+                    <origin rpy="3.14 0 -1.570" xyz="0.006 -0.005 -0.034"/>
+                </xacro:if>
+                <xacro:unless value="${(mirror == False)}">
+                    <origin rpy="3.14 0 -1.570" xyz="0.006 0.005 -0.034"/>
+                </xacro:unless>
                 <geometry>
-                    <mesh filename="package://legged_unitree_description/meshes/$(arg robot_type)/${prefix}_ShoulderRx.dae"
+                    <mesh filename="package://legged_unitree_description/meshes/$(arg robot_type)/L_ShoulderRx.obj"
                             scale="1 1 1"/>
                 </geometry>
-                <material name="orange"/>
+                <material name="red"/>
             </visual>
             <inertial>
@@ -41,11 +46,11 @@
             <visual>
             <xacro:if value="${(mirror == True)}">
-                <origin rpy="0 0 -3.14" xyz="0. 0.0 0"/>
+                <origin rpy="1.57 1.57 0" xyz="0. 0.07 0.02"/>
             </xacro:if>
-            <xacro:if value="${(mirror == False)}">
-                <origin rpy="0 0 0.0" xyz="0 0 0.0"/>
-            </xacro:if>
+            <xacro:unless value="${(mirror == False)}">
+                <origin rpy="1.57 1.57 0.0" xyz="0 -0.07 0.02"/>
+            </xacro:unless>
                 <geometry>
-                    <mesh filename="package://legged_unitree_description/meshes/$(arg robot_type)/${prefix}_UpperArm.dae"
+                    <mesh filename="package://legged_unitree_description/meshes/$(arg robot_type)/${prefix}_UpperArm.obj"
                             scale="1 1 1"/>
                 </geometry>
@@ -72,7 +77,25 @@
         <link name="${prefix}_LForeArm">
             <visual>
-                <origin rpy="0 0 0.0" xyz="0. 0 0"/>
+                <xacro:if value="${(mirror == True)}">
+                    <origin rpy="0 0 0" xyz="-0.05 -0.075 0.16"/>
+                </xacro:if>
+                <xacro:unless value="${(mirror == False)}">
+                    <origin rpy="0 0 3.14" xyz="-0.05 0.075 0.16"/>
+                </xacro:unless>
                 <geometry>
-                    <mesh filename="package://legged_unitree_description/meshes/$(arg robot_type)/${prefix}_ForeArm2.dae"
+                    <mesh filename="package://legged_unitree_description/meshes/$(arg robot_type)/R_ShoulderRx.obj"
+                            scale="1 1 1"/>
+                </geometry>
+                <material name="orange"/>
+            </visual>
+            <visual>
+                <xacro:if value="${(mirror == True)}">
+                    <origin rpy="0 1.570 0.0" xyz="-0.0 -0.0 0.0"/>
+                </xacro:if>
+                <xacro:unless value="${(mirror == False)}">
+                    <origin rpy="0 1.570 0.0" xyz="-0.0 0.0 -0.102"/>
+                </xacro:unless>
+                <geometry>
+                    <mesh filename="package://legged_unitree_description/meshes/$(arg robot_type)/${prefix}_ForeArm2.obj"
                             scale="1 1 1"/>
                 </geometry>

File: src/legged_examples/legged_unitree/legged_unitree_description/urdf/common/leg.xacro (robot description, xacro)
@@ -15,5 +15,5 @@
                 <origin rpy="0 0 0.0" xyz="0 0 0"/>
                 <geometry>
-                    <mesh filename="package://legged_unitree_description/meshes/$(arg robot_type)/${prefix}_HipRz.dae"
+                    <mesh filename="package://legged_unitree_description/meshes/$(arg robot_type)/${prefix}_HipRz.obj"
                             scale="1 1 1"/>
                 </geometry>
@@ -40,7 +40,12 @@
         <link name="${prefix}_LHipRx">
             <visual>
-                <origin rpy="0 -1.57 0.0" xyz="0 0 0"/>
-                <geometry>
-                    <mesh filename="package://legged_unitree_description/meshes/$(arg robot_type)/${prefix}_HipRx.dae"
+                <xacro:if value="${(mirror == True)}">
+                    <origin rpy="0 -3.14 -3.14" xyz="0. 0.00 -0.0"/>
+                </xacro:if>
+                <xacro:if value="${(mirror == False)}">
+                    <origin rpy="0 0 0.0" xyz="0 0 0.0"/>
+                </xacro:if>
+                <geometry>
+                    <mesh filename="package://legged_unitree_description/meshes/$(arg robot_type)/${prefix}_HipRx.obj"
                             scale="1 1 1"/>
                 </geometry>
@@ -67,7 +72,12 @@
         <link name="${prefix}_LThigh">
             <visual>
-                <origin rpy="0 1.57 -1.57" xyz="0 0 0"/>
-                <geometry>
-                    <mesh filename="package://legged_unitree_description/meshes/$(arg robot_type)/${prefix}_Thigh.dae"
+                <xacro:if value="${(mirror == True)}">
+                    <origin rpy="0 0 -3.14" xyz="0. 0.00 -0.0"/>
+                </xacro:if>
+                <xacro:if value="${(mirror == False)}">
+                    <origin rpy="0 0 0.0" xyz="0 0 0.0"/>
+                </xacro:if>
+                <geometry>
+                    <mesh filename="package://legged_unitree_description/meshes/$(arg robot_type)/${prefix}_Thigh.obj"
                             scale="1 1 1"/>
                 </geometry>
@@ -94,7 +104,7 @@
         <link name="${prefix}_LShank">
             <visual>
-                <origin rpy="1.57 1.57 0" xyz="0 0 0"/>
-                <geometry>
-                    <mesh filename="package://legged_unitree_description/meshes/$(arg robot_type)/${prefix}_LowerLeg3_drawing.dae"
+                <origin rpy="0 -3.14 0" xyz="0 -0.6 0"/>
+                <geometry>
+                    <mesh filename="package://legged_unitree_description/meshes/$(arg robot_type)/${prefix}_LowerLeg3_drawing.obj"
                             scale="1 1 1"/>
                 </geometry>
@@ -123,5 +133,5 @@
                 <origin rpy="1.57 1.57 0" xyz="0 0 0"/>
                 <geometry>
-                    <mesh filename="package://legged_unitree_description/meshes/$(arg robot_type)/${prefix}_foot_drawing.dae"
+                    <mesh filename="package://legged_unitree_description/meshes/$(arg robot_type)/${prefix}_foot_drawing.obj"
                             scale="1 1 1"/>
                 </geometry>

File: src/legged_examples/legged_unitree/legged_unitree_description/urdf/robot.xacro (robot description, xacro)
@@ -12,5 +12,5 @@
             <origin rpy="0 0 0" xyz="0 0 0"/>
             <geometry>
-                <mesh filename="package://legged_unitree_description/meshes/$(arg robot_type)/Body.dae" scale="1 1 1"/>
+                <mesh filename="package://legged_unitree_description/meshes/$(arg robot_type)/Body.obj" scale="1 1 1"/>
             </geometry>
         </visual>

Commit message: comment something

File: src/legged_examples/legged_unitree/legged_unitree_description/urdf/common/arm.xacro (robot description, xacro)
@@ -51,5 +51,5 @@
             <axis xyz="0 1 0"/>
             <dynamics damping="${damping}" friction="${friction}"/>
-            <limit effort="${hip_torque_max}" velocity="${hip_torque_max}" lower="${hip_min}"
+            <limit effort="${hip_torque_max}" velocity="${hip_velocity_max}" lower="${hip_min}"
                    upper="${hip_max}"/>
         </joint>
@@ -94,5 +94,5 @@
             <axis xyz="0 1 0"/>
             <dynamics damping="${damping}" friction="${friction}"/>
-            <limit effort="${hip_torque_max}" velocity="${hip_torque_max}" lower="${hip_min}"
+            <limit effort="${hip_torque_max}" velocity="${hip_velocity_max}" lower="${hip_min}"
                    upper="${hip_max}"/>
         </joint>

File: src/legged_examples/legged_unitree/legged_unitree_description/urdf/common/leg.xacro (robot description, xacro)
@@ -159,5 +159,5 @@
             <axis xyz="0 1 0"/>
             <dynamics damping="${damping}" friction="${friction}"/>
-            <limit effort="${hip_torque_max}" velocity="${hip_velocity_max}" lower="${hip_min}"
+            <limit effort="${hip_torque_max}" velocity="${hip_max}" lower="${hip_min}"
                    upper="${hip_max}"/>
         </joint>
