Commit message: edit --> legged_unitree_description

File: src/legged_examples/legged_unitree/legged_unitree_description/urdf/a1/const.xacro (robot description, xacro)
@@ -45,14 +45,14 @@
     <!-- dynamics inertial value -->
     <!-- trunk -->
-    <xacro:property name="trunk_mass" value="6.0"/>
+    <xacro:property name="trunk_mass" value="6.5"/>
     <xacro:property name="trunk_com_x" value="0.0000"/>
-    <xacro:property name="trunk_com_y" value="0.0041"/>
-    <xacro:property name="trunk_com_z" value="-0.0005"/>
-    <xacro:property name="trunk_ixx" value="0.0158533"/>
-    <xacro:property name="trunk_ixy" value="-0.0000366"/>
-    <xacro:property name="trunk_ixz" value="-0.0000611"/>
-    <xacro:property name="trunk_iyy" value="0.0377999"/>
-    <xacro:property name="trunk_iyz" value="-0.0000275"/>
-    <xacro:property name="trunk_izz" value="0.0456542"/>
+    <xacro:property name="trunk_com_y" value="0.0"/>
+    <xacro:property name="trunk_com_z" value="0.15"/>
+    <xacro:property name="trunk_ixx" value="0.3006167"/>
+    <xacro:property name="trunk_ixy" value="-0.0"/>
+    <xacro:property name="trunk_ixz" value="-0.0"/>
+    <xacro:property name="trunk_iyy" value="0.23837"/>
+    <xacro:property name="trunk_iyz" value="-0.0"/>
+    <xacro:property name="trunk_izz" value="0.09690467"/>
     <!-- hip (left front) -->
     <xacro:property name="hip_mass" value="0.595"/>

File: src/legged_examples/legged_unitree/legged_unitree_description/urdf/common/leg.xacro (robot description, xacro)
@@ -5,5 +5,4 @@
         <joint name="${prefix}_JHipRz" type="revolute">
             <xacro:insert_block name="origin"/>
-            <origin rpy="0 0 0" xyz="0 ${0.075*mirror} 0"/>
             <parent link="base"/>
             <child link="${prefix}_LHipRz"/>

File: src/legged_examples/legged_unitree/legged_unitree_description/urdf/common/transmission.xacro (robot description, xacro)
@@ -2,30 +2,50 @@
 <robot xmlns:xacro="http://www.ros.org/wiki/xacro">
     <xacro:macro name="leg_transmission" params="name">
-        <transmission name="${prefix}_HAA_tran">
+        <transmission name="${prefix}_JHipRz_tran">
             <type>transmission_interface/SimpleTransmission</type>
-            <joint name="${prefix}_HAA">
+            <joint name="${prefix}_JHipRz">
                 <hardwareInterface>hardware_interface/EffortJointInterface</hardwareInterface>
             </joint>
-            <actuator name="${prefix}_HAA_motor">
+            <actuator name="${prefix}_JHipRz_motor">
                 <hardwareInterface>hardware_interface/EffortJointInterface</hardwareInterface>
                 <mechanicalReduction>1</mechanicalReduction>
             </actuator>
         </transmission>
-        <transmission name="${prefix}_HFE_tran">
+        <transmission name="${prefix}_JHipRx_tran">
             <type>transmission_interface/SimpleTransmission</type>
-            <joint name="${prefix}_HFE">
+            <joint name="${prefix}_JHipRx">
                 <hardwareInterface>hardware_interface/EffortJointInterface</hardwareInterface>
             </joint>
-            <actuator name="${prefix}_HFE_motor">
+            <actuator name="${prefix}_JHipRx_motor">
                 <hardwareInterface>hardware_interface/EffortJointInterface</hardwareInterface>
                 <mechanicalReduction>1</mechanicalReduction>
             </actuator>
         </transmission>
-        <transmission name="${prefix}_KFE_tran">
+        <transmission name="${prefix}_JThigh_tran">
             <type>transmission_interface/SimpleTransmission</type>
-            <joint name="${prefix}_KFE">
+            <joint name="${prefix}_JThigh">
                 <hardwareInterface>hardware_interface/EffortJointInterface</hardwareInterface>
             </joint>
-            <actuator name="${prefix}_KFE_motor">
+            <actuator name="${prefix}_JThigh_motor">
+                <hardwareInterface>hardware_interface/EffortJointInterface</hardwareInterface>
+                <mechanicalReduction>1</mechanicalReduction>
+            </actuator>
+        </transmission>
+        <transmission name="${prefix}_JKnee_tran">
+            <type>transmission_interface/SimpleTransmission</type>
+            <joint name="${prefix}_JKnee">
+                <hardwareInterface>hardware_interface/EffortJointInterface</hardwareInterface>
+            </joint>
+            <actuator name="${prefix}_JKnee_motor">
+                <hardwareInterface>hardware_interface/EffortJointInterface</hardwareInterface>
+                <mechanicalReduction>1</mechanicalReduction>
+            </actuator>
+        </transmission>
+        <transmission name="${prefix}_JAnkle_tran">
+            <type>transmission_interface/SimpleTransmission</type>
+            <joint name="${prefix}_JAnkle">
+                <hardwareInterface>hardware_interface/EffortJointInterface</hardwareInterface>
+            </joint>
+            <actuator name="${prefix}_JAnkle_motor">
                 <hardwareInterface>hardware_interface/EffortJointInterface</hardwareInterface>
                 <mechanicalReduction>1</mechanicalReduction>

File: src/legged_examples/legged_unitree/legged_unitree_description/urdf/robot.xacro (robot description, xacro)
@@ -4,4 +4,5 @@
     <xacro:include filename="$(find legged_unitree_description)/urdf/common/materials.xacro"/>
     <xacro:include filename="$(find legged_unitree_description)/urdf/common/leg.xacro"/>
+    <xacro:include filename="$(find legged_unitree_description)/urdf/common/arm.xacro"/>
     <xacro:include filename="$(find legged_unitree_description)/urdf/common/gazebo.xacro"/>
     <xacro:include filename="$(find legged_unitree_description)/urdf/common/imu.xacro"/>
@@ -31,8 +32,14 @@
     <xacro:IMU connected_to="base" imu_name="unitree_imu" xyz="0. 0. 0." rpy="0. 0. 0."/>
     <xacro:leg prefix="L" mirror="1" mirror_dae="False" front_hind="1" front_hind_dae="True">
-        <origin rpy="0 0 0" xyz="${leg_offset_x} ${-leg_offset_y} 0"/>
+        <origin rpy="0 0 0" xyz="0 0.075 0"/>
     </xacro:leg>
     <xacro:leg prefix="R" mirror="-1" mirror_dae="True" front_hind="1" front_hind_dae="True">
-        <origin rpy="0 0 0" xyz="${leg_offset_x} ${leg_offset_y} 0"/>
+        <origin rpy="0 0 0" xyz="0 -0.075 0"/>
+    </xacro:leg>
+    <xacro:arm prefix="L" mirror="1" mirror_dae="False" front_hind="1" front_hind_dae="True">
+        <origin rpy="0 0 0" xyz="-0.0215 0.1115 0.202"/>
+    </xacro:leg>
+    <xacro:arm prefix="R" mirror="-1" mirror_dae="True" front_hind="1" front_hind_dae="True">
+        <origin rpy="0 0 0" xyz="-0.0215 -0.1115 0.202"/>
     </xacro:leg>
 </robot>

Commit message: file: urdf frame correct

File: src/legged_examples/legged_unitree/legged_unitree_description/urdf/a1/const.xacro (robot description, xacro)
@@ -29,8 +29,8 @@
     <xacro:property name="hip_offset" value="0.065"/>
     <!-- joint limits -->
-    <xacro:property name="damping" value="0"/>
-    <xacro:property name="friction" value="0"/>
-    <xacro:property name="hip_max" value="${46*pi/180.0}"/>
-    <xacro:property name="hip_min" value="${-46*pi/180.0}"/>
+    <xacro:property name="damping" value="100"/>
+    <xacro:property name="friction" value="100"/>
+    <xacro:property name="hip_max" value="3"/>
+    <xacro:property name="hip_min" value="-3"/>
     <xacro:property name="hip_velocity_max" value="21"/>
     <xacro:property name="hip_torque_max" value="33.5"/>

File: src/legged_examples/legged_unitree/legged_unitree_description/urdf/a2.urdf (robot description, URDF)
Before this commit: robot robot, 18 links, 17 joints
Joints:
- joint L_JAnkle: limit lower=-0.8028514559173915 upper=-0.8028514559173915 effort=33.5 velocity=33.5 -> lower=-3 upper=3 effort=33.5 velocity=33.5
- joint L_JForeArm: limit lower=-0.8028514559173915 upper=-0.8028514559173915 effort=33.5 velocity=33.5 -> lower=-3 upper=3 effort=33.5 velocity=33.5
- joint L_JHipRx: limit lower=-0.8028514559173915 upper=-0.8028514559173915 effort=33.5 velocity=33.5 -> lower=-3 upper=3 effort=33.5 velocity=33.5
- joint L_JHipRz: limit lower=-0.8028514559173915 upper=0.8028514559173915 effort=33.5 velocity=21 -> lower=-3 upper=3 effort=33.5 velocity=21
- joint L_JKnee: limit lower=-0.8028514559173915 upper=-0.8028514559173915 effort=33.5 velocity=33.5 -> lower=-3 upper=3 effort=33.5 velocity=33.5
- joint L_JShoulderRx: limit lower=-0.8028514559173915 upper=0.8028514559173915 effort=33.5 velocity=21 -> lower=-3 upper=3 effort=33.5 velocity=21
- joint L_JThigh: limit lower=-0.8028514559173915 upper=-0.8028514559173915 effort=33.5 velocity=33.5 -> lower=-3 upper=3 effort=33.5 velocity=33.5
- joint L_JUpperArm: limit lower=-0.8028514559173915 upper=-0.8028514559173915 effort=33.5 velocity=33.5 -> lower=-3 upper=3 effort=33.5 velocity=33.5
- joint R_JAnkle: limit lower=-0.8028514559173915 upper=-0.8028514559173915 effort=33.5 velocity=33.5 -> lower=-3 upper=3 effort=33.5 velocity=33.5
- joint R_JForeArm: limit lower=-0.8028514559173915 upper=-0.8028514559173915 effort=33.5 velocity=33.5 -> lower=-3 upper=3 effort=33.5 velocity=33.5
- joint R_JHipRx: limit lower=-0.8028514559173915 upper=-0.8028514559173915 effort=33.5 velocity=33.5 -> lower=-3 upper=3 effort=33.5 velocity=33.5
- joint R_JHipRz: limit lower=-0.8028514559173915 upper=0.8028514559173915 effort=33.5 velocity=21 -> lower=-3 upper=3 effort=33.5 velocity=21
- joint R_JKnee: limit lower=-0.8028514559173915 upper=-0.8028514559173915 effort=33.5 velocity=33.5 -> lower=-3 upper=3 effort=33.5 velocity=33.5
- joint R_JShoulderRx: limit lower=-0.8028514559173915 upper=0.8028514559173915 effort=33.5 velocity=21 -> lower=-3 upper=3 effort=33.5 velocity=21
- joint R_JThigh: limit lower=-0.8028514559173915 upper=-0.8028514559173915 effort=33.5 velocity=33.5 -> lower=-3 upper=3 effort=33.5 velocity=33.5
- joint R_JUpperArm: limit lower=-0.8028514559173915 upper=-0.8028514559173915 effort=33.5 velocity=33.5 -> lower=-3 upper=3 effort=33.5 velocity=33.5

File: src/legged_examples/legged_unitree/legged_unitree_description/urdf/common/arm.xacro (robot description, xacro)
@@ -36,5 +36,5 @@
             <dynamics damping="${damping}" friction="${friction}"/>
             <limit effort="${hip_torque_max}" velocity="${hip_torque_max}" lower="${hip_min}"
-                   upper="${hip_min}"/>
+                   upper="${hip_max}"/>
         </joint>
         <link name="${prefix}_LUpperArm">
@@ -63,5 +63,5 @@
             <dynamics damping="${damping}" friction="${friction}"/>
             <limit effort="${hip_torque_max}" velocity="${hip_torque_max}" lower="${hip_min}"
-                   upper="${hip_min}"/>
+                   upper="${hip_max}"/>
         </joint>
         <link name="${prefix}_LForeArm">

File: src/legged_examples/legged_unitree/legged_unitree_description/urdf/common/leg.xacro (robot description, xacro)
@@ -36,5 +36,5 @@
             <dynamics damping="${damping}" friction="${friction}"/>
             <limit effort="${hip_torque_max}" velocity="${hip_torque_max}" lower="${hip_min}"
-                   upper="${hip_min}"/>
+                   upper="${hip_max}"/>
         </joint>
         <link name="${prefix}_LHipRx">
@@ -63,5 +63,5 @@
             <dynamics damping="${damping}" friction="${friction}"/>
             <limit effort="${hip_torque_max}" velocity="${hip_torque_max}" lower="${hip_min}"
-                   upper="${hip_min}"/>
+                   upper="${hip_max}"/>
         </joint>
         <link name="${prefix}_LThigh">
@@ -90,5 +90,5 @@
             <dynamics damping="${damping}" friction="${friction}"/>
             <limit effort="${hip_torque_max}" velocity="${hip_torque_max}" lower="${hip_min}"
-                   upper="${hip_min}"/>
+                   upper="${hip_max}"/>
         </joint>
         <link name="${prefix}_LShank">
@@ -117,5 +117,5 @@
             <dynamics damping="${damping}" friction="${friction}"/>
             <limit effort="${hip_torque_max}" velocity="${hip_torque_max}" lower="${hip_min}"
-                   upper="${hip_min}"/>
+                   upper="${hip_max}"/>
         </joint>
         <link name="${prefix}_Foot">
