Commit message: add collision in leg.xacro

File: src/legged_examples/legged_unitree/legged_unitree_description/urdf/a1/const.xacro (robot description, xacro)
@@ -3,20 +3,45 @@
     <!-- Constants for robot dimensions -->
     <xacro:property name="stick_mass" value="0.00001"/>
+    <!-- <xacro:property name="trunk_width" value="0.08"/>
+    <xacro:property name="trunk_length" value="0.22"/>
+    <xacro:property name="trunk_height" value="0.14"/> -->
     <!-- simplified collision value -->
     <xacro:property name="trunk_width" value="0.194"/>
     <xacro:property name="trunk_length" value="0.267"/>
-    <xacro:property name="trunk_height" value="0.114"/>
-    <xacro:property name="hip_radius" value="0.046"/>
-    <xacro:property name="hip_length" value="0.04"/>
-    <xacro:property name="thigh_shoulder_radius" value="0.041"/>
-    <xacro:property name="thigh_shoulder_length" value="0.04"/>
-    <xacro:property name="thigh_shoulder_y_offset" value="-0.008"/>
-    <xacro:property name="thigh_width" value="0.03"/>
-    <xacro:property name="thigh_height" value="0.034"/>
-    <xacro:property name="thigh_x_offset" value="-0.015"/>
-    <xacro:property name="calf_width" value="0.016"/>
-    <xacro:property name="calf_height" value="0.016"/>
-    <xacro:property name="calf_x_offset" value="0.0"/>
-    <xacro:property name="foot_radius" value="0.02"/>
+    <xacro:property name="trunk_height" value="0.178"/>
+    <xacro:property name="shoudlerarm_radius" value="0.05"/>
+    <xacro:property name="shoudlerarm_length" value="0.02"/>
+    <xacro:property name="shoudlerarm_x_offset" value="-0.05"/>
+    <xacro:property name="shoudlerarm_y_offset" value="0.0"/>
+    <xacro:property name="shoudlerarm_z_offset" value="-0.0"/>
+    <xacro:property name="shoudlerarm_ry_offset" value="1.57"/>
+    <xacro:property name="upperarm_radius" value="0.025"/>
+    <xacro:property name="upperarm_length" value="0.23"/>
+    <xacro:property name="upperarm_x_offset" value="0.01"/>
+    <xacro:property name="upperarm_y_offset" value="0.068"/>
+    <xacro:property name="upperarm_z_offset" value="-0.05"/>
+    <xacro:property name="forearm_radius" value="0.025"/>
+    <xacro:property name="forearm_length" value="0.23"/>
+    <xacro:property name="forearm_x_offset" value="0.015"/>
+    <xacro:property name="forearm_y_offset" value="0.007"/>
+    <xacro:property name="forearm_z_offset" value="-0.1"/>
+    <xacro:property name="HipRx_radius" value="0.04"/>
+    <xacro:property name="HipRx_length" value="0.05"/>
+    <xacro:property name="HipRx_x_offset" value="-0.07"/>
+    <xacro:property name="HipRx_y_offset" value="-0.0"/>
+    <xacro:property name="HipRx_z_offset" value="-0.0"/>
+    <xacro:property name="HipRx_ry_offset" value="1.57"/>
+    <xacro:property name="Shank_radius" value="0.04"/>
+    <xacro:property name="Shank_length" value="0.2"/>
+    <xacro:property name="Shank_x_offset" value="-0.0"/>
+    <xacro:property name="Shank_y_offset" value="-0.0"/>
+    <xacro:property name="Shank_z_offset" value="-0.15"/>
+    <xacro:property name="Shank_ry_offset" value="0"/>
+    <xacro:property name="Thigh_radius" value="0.04"/>
+    <xacro:property name="Thigh_length" value="0.23"/>
+    <xacro:property name="Thigh_x_offset" value="-0.0"/>
+    <xacro:property name="Thigh_y_offset" value="-0.0"/>
+    <xacro:property name="Thigh_z_offset" value="-0.17"/>
+    <xacro:property name="Thigh_ry_offset" value="0"/>
     <!-- kinematic value -->
     <xacro:property name="thigh_offset" value="0.0838"/>

File: src/legged_examples/legged_unitree/legged_unitree_description/urdf/common/arm.xacro (robot description, xacro)
@@ -25,4 +25,15 @@
                 <material name="red"/>
             </visual>
+            <collision>
+            <xacro:if value="${(mirror == True)}">
+                <origin rpy="0 ${shoudlerarm_ry_offset} 0" xyz="${shoudlerarm_x_offset} ${shoudlerarm_y_offset} ${shoudlerarm_z_offset}"/>
+            </xacro:if>
+            <xacro:unless value="${(mirror == False)}">
+                <origin rpy="0 ${shoudlerarm_ry_offset} 0" xyz="${shoudlerarm_x_offset} ${-shoudlerarm_y_offset} ${shoudlerarm_z_offset}"/>
+            </xacro:unless>
+                <geometry>
+                    <cylinder length="${shoudlerarm_length}" radius="${shoudlerarm_radius}"/>
+                </geometry>
+            </collision>
             <inertial>
                 <origin rpy="0 0 0" xyz="0.01 0.0 0.0"/>
@@ -57,4 +68,15 @@
                 <material name="orange"/>
             </visual>
+            <collision>
+            <xacro:if value="${(mirror == True)}">
+                <origin rpy="0 0 0" xyz="${upperarm_x_offset} ${upperarm_y_offset} ${upperarm_z_offset}"/>
+            </xacro:if>
+            <xacro:unless value="${(mirror == False)}">
+                <origin rpy="0 0 0" xyz="${upperarm_x_offset} ${-upperarm_y_offset} ${upperarm_z_offset}"/>
+            </xacro:unless>
+                <geometry>
+                    <cylinder length="${upperarm_length}" radius="${upperarm_radius}"/>
+                </geometry>
+            </collision>
             <inertial>
                 <origin rpy="0 0 0" xyz="0.0 0.0 -0.09"/>
@@ -102,4 +124,15 @@
                 <material name="orange"/>
             </visual>
+            <collision>
+            <xacro:if value="${(mirror == True)}">
+                <origin rpy="0 0 0" xyz="${forearm_x_offset} ${forearm_y_offset} ${forearm_z_offset}"/>
+            </xacro:if>
+            <xacro:unless value="${(mirror == False)}">
+                <origin rpy="0 0 0" xyz="${forearm_x_offset} ${-forearm_y_offset} ${forearm_z_offset}"/>
+            </xacro:unless>
+                <geometry>
+                    <cylinder length="${forearm_length}" radius="${forearm_radius}"/>
+                </geometry>
+            </collision>
             <inertial>
                 <origin rpy="0 0 0" xyz="0.0 0.0 -0.04"/>

File: src/legged_examples/legged_unitree/legged_unitree_description/urdf/common/leg.xacro (robot description, xacro)
@@ -39,4 +39,15 @@
         </joint>
         <link name="${prefix}_LHipRx">
+            <collision>
+            <xacro:if value="${(mirror == True)}">
+                <origin rpy="0 ${HipRx_ry_offset} 0" xyz="${HipRx_x_offset} ${HipRx_y_offset} ${HipRx_z_offset}"/>
+            </xacro:if>
+            <xacro:unless value="${(mirror == False)}">
+                <origin rpy="0 ${HipRx_ry_offset} 0" xyz="${HipRx_x_offset} ${-HipRx_y_offset} ${HipRx_z_offset}"/>
+            </xacro:unless>
+                <geometry>
+                    <cylinder length="${HipRx_length}" radius="${HipRx_radius}"/>
+                </geometry>
+            </collision>
             <visual>
                 <xacro:if value="${(mirror == True)}">
@@ -84,4 +95,15 @@
                 <material name="orange"/>
             </visual>
+            <collision>
+            <xacro:if value="${(mirror == True)}">
+                <origin rpy="0 0 0" xyz="${Thigh_x_offset} ${Thigh_y_offset} ${Thigh_z_offset}"/>
+            </xacro:if>
+            <xacro:unless value="${(mirror == False)}">
+                <origin rpy="0 0 0" xyz="${Thigh_x_offset} ${-Thigh_y_offset} ${Thigh_z_offset}"/>
+            </xacro:unless>
+                <geometry>
+                    <cylinder length="${Thigh_length}" radius="${Thigh_radius}"/>
+                </geometry>
+            </collision>
             <inertial>
                 <origin rpy="0 0 0" xyz="0.0 0.0 -0.01"/>
@@ -111,4 +133,15 @@
                 <material name="orange"/>
             </visual>
+            <collision>
+            <xacro:if value="${(mirror == True)}">
+                <origin rpy="0 0 0" xyz="${Shank_x_offset} ${Shank_y_offset} ${Shank_z_offset}"/>
+            </xacro:if>
+            <xacro:unless value="${(mirror == False)}">
+                <origin rpy="0 0 0" xyz="${Shank_x_offset} ${-Shank_y_offset} ${Shank_z_offset}"/>
+            </xacro:unless>
+                <geometry>
+                    <cylinder length="${Shank_length}" radius="${Shank_radius}"/>
+                </geometry>
+            </collision>
             <inertial>
                 <origin rpy="0 0 0" xyz="-0.03416 -0.00075 -0.01"/>
@@ -138,9 +171,21 @@
                 <material name="orange"/>
             </visual>
-            <visual>
+            <!-- <visual>
                 <geometry>
                     <sphere radius="0.001"/>
                 </geometry>
                 <origin xyz="0.125 0.0 -0.033" rpy="0 0 0"/>
+            </visual> -->
+            <collision>
+                <geometry>
+                    <sphere radius="0.02"/>
+                </geometry>
+                <origin xyz="0 0.0 -0.033" rpy="0 0 0"/>
+            </collision>
+            <!-- <visual>
+                <geometry>
+                    <sphere radius="0.001"/>
+                </geometry>
+                <origin xyz="-0.025 0.0 -0.033" rpy="0 0 0"/>
             </visual>
             <collision>
@@ -148,18 +193,6 @@
                     <sphere radius="0.0"/>
                 </geometry>
-                <origin xyz="0.125 0.0 -0.033" rpy="0 0 0"/>
-            </collision>
-            <visual>
-                <geometry>
-                    <sphere radius="0.001"/>
-                </geometry>
                 <origin xyz="-0.025 0.0 -0.033" rpy="0 0 0"/>
-            </visual>
-            <collision>
-                <geometry>
-                    <sphere radius="0.0"/>
-                </geometry>
-                <origin xyz="-0.025 0.0 -0.033" rpy="0 0 0"/>
-            </collision>
+            </collision> -->
             <inertial>
                 <origin rpy="0 0 0" xyz="0.0 0.0 -0.01"/>

File: src/legged_examples/legged_unitree/legged_unitree_description/urdf/robot.urdf (robot description, URDF)
Before this commit: robot robot, 18 links, 17 joints
Links:
- link L_Foot: geometry collision sphere radius=0.02; visual mesh filename=package://legged_unitree_description/meshes/a1/L_foot_drawi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 scale=1 1 1
- link L_LForeArm: geometry collision cylinder length=0.23 radius=0.025; visual mesh filename=package://legged_unitree_description/meshes/a1/L_ForeArm2.o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 scale=1 1 1
- link L_LHipRx: geometry collision cylinder length=0.05 radius=0.04; visual mesh filename=package://legged_unitree_description/meshes/a1/L_HipRx.obj scale=1 1 1
- link L_LShank: geometry collision cylinder length=0.2 radius=0.04; visual mesh filename=package://legged_unitree_description/meshes/a1/L_LowerLeg3_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 scale=1 1 1
- link L_LShoulderRx: geometry collision cylinder length=0.02 radius=0.05; visual mesh filename=package://legged_unitree_description/meshes/a1/L_ShoulderRx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 scale=1 1 1
- link L_LThigh: geometry collision cylinder length=0.23 radius=0.04; visual mesh filename=package://legged_unitree_description/meshes/a1/L_Thigh.obj scale=1 1 1
- link L_LUpperArm: geometry collision cylinder length=0.23 radius=0.025; visual mesh filename=package://legged_unitree_description/meshes/a1/L_UpperArm.o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 scale=1 1 1
- link R_Foot: geometry collision sphere radius=0.02; visual mesh filename=package://legged_unitree_description/meshes/a1/R_foot_drawi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 scale=1 1 1
- link R_LForeArm: geometry collision cylinder length=0.23 radius=0.025; visual mesh filename=package://legged_unitree_description/meshes/a1/R_ForeArm2.o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 scale=1 1 1
- link R_LHipRx: geometry collision cylinder length=0.05 radius=0.04; visual mesh filename=package://legged_unitree_description/meshes/a1/R_HipRx.obj scale=1 1 1
- link R_LShank: geometry collision cylinder length=0.2 radius=0.04; visual mesh filename=package://legged_unitree_description/meshes/a1/R_LowerLeg3_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 scale=1 1 1
- link R_LShoulderRx: geometry collision cylinder length=0.02 radius=0.05; visual mesh filename=package://legged_unitree_description/meshes/a1/L_ShoulderRx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 scale=1 1 1
- link R_LThigh: geometry collision cylinder length=0.23 radius=0.04; visual mesh filename=package://legged_unitree_description/meshes/a1/R_Thigh.obj scale=1 1 1
- link R_LUpperArm: geometry collision cylinder length=0.23 radius=0.025; visual mesh filename=package://legged_unitree_description/meshes/a1/R_UpperArm.o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 scale=1 1 1
- link base: geometry collision box size=0.194 0.267 0.178; visual mesh filename=package://legged_unitree_description/meshes/a1/Body.obj scale=1 1 1

File: src/legged_examples/legged_unitree/legged_unitree_description/urdf/robot.xacro (robot description, xacro)
@@ -16,7 +16,7 @@
         </visual>
         <collision>
-            <origin rpy="0 0 0" xyz="0 0 0"/>
+            <origin rpy="0 0 0" xyz="0 0 0.04"/>
             <geometry>
-                <box size="${trunk_length} ${trunk_width} ${trunk_height}"/>
+                <box size="${trunk_width} ${trunk_length} ${trunk_height}"/>
             </geometry>
         </collision>

Commit message: correct foot collision

File: src/legged_examples/legged_unitree/legged_unitree_description/urdf/a1/const.xacro (robot description, xacro)
@@ -44,4 +44,7 @@
     <xacro:property name="Thigh_z_offset" value="-0.17"/>
     <xacro:property name="Thigh_ry_offset" value="0"/>
+    <xacro:property name="foot_width" value="0.16"/>
+    <xacro:property name="foot_length" value="0.042"/>
+    <xacro:property name="foot_height" value="0.016"/>
     <!-- kinematic value -->
     <xacro:property name="thigh_offset" value="0.0838"/>

File: src/legged_examples/legged_unitree/legged_unitree_description/urdf/common/leg.xacro (robot description, xacro)
@@ -35,5 +35,5 @@
             <axis xyz="1 0 0"/>
             <dynamics damping="${damping}" friction="${friction}"/>
-            <limit effort="${hip_torque_max}" velocity="${hip_torque_max}" lower="${hip_min}"
+            <limit effort="${hip_torque_max}" velocity="${hip_velocity_max}" lower="${hip_min}"
                    upper="${hip_max}"/>
         </joint>
@@ -78,5 +78,5 @@
             <axis xyz="0 1 0"/>
             <dynamics damping="${damping}" friction="${friction}"/>
-            <limit effort="${hip_torque_max}" velocity="${hip_torque_max}" lower="${hip_min}"
+            <limit effort="${hip_torque_max}" velocity="${hip_velocity_max}" lower="${hip_min}"
                    upper="${hip_max}"/>
         </joint>
@@ -121,5 +121,5 @@
             <axis xyz="0 1 0"/>
             <dynamics damping="${damping}" friction="${friction}"/>
-            <limit effort="${hip_torque_max}" velocity="${hip_torque_max}" lower="${hip_min}"
+            <limit effort="${hip_torque_max}" velocity="${hip_velocity_max}" lower="${hip_min}"
                    upper="${hip_max}"/>
         </joint>
@@ -159,5 +159,5 @@
             <axis xyz="0 1 0"/>
             <dynamics damping="${damping}" friction="${friction}"/>
-            <limit effort="${hip_torque_max}" velocity="${hip_torque_max}" lower="${hip_min}"
+            <limit effort="${hip_torque_max}" velocity="${hip_velocity_max}" lower="${hip_min}"
                    upper="${hip_max}"/>
         </joint>
@@ -177,10 +177,10 @@
                 <origin xyz="0.125 0.0 -0.033" rpy="0 0 0"/>
             </visual> -->
-            <collision>
+            <!-- <collision>
                 <geometry>
                     <sphere radius="0.02"/>
                 </geometry>
-                <origin xyz="0 0.0 -0.033" rpy="0 0 0"/>
-            </collision>
+                <origin xyz="0.01 0.0 -0.033" rpy="0 0 0"/>
+            </collision> -->
             <!-- <visual>
                 <geometry>
@@ -188,11 +188,28 @@
                 </geometry>
                 <origin xyz="-0.025 0.0 -0.033" rpy="0 0 0"/>
-            </visual>
-            <collision>
-                <geometry>
-                    <sphere radius="0.0"/>
-                </geometry>
-                <origin xyz="-0.025 0.0 -0.033" rpy="0 0 0"/>
+            </visual>-->
+            <!-- <collision>
+                <geometry>
+                    <sphere radius="0.02"/>
+                </geometry>
+                <origin xyz="-0.01 0.0 -0.033" rpy="0 0 0"/>
+            </collision>  -->
+            <!-- <collision>
+            <xacro:if value="${(mirror == True)}">
+                <origin rpy="0 0 0" xyz="${foot_width} ${Shank_y_offset} ${Shank_z_offset}"/>
+            </xacro:if>
+            <xacro:unless value="${(mirror == False)}">
+                <origin rpy="0 0 0" xyz="${Shank_x_offset} ${-Shank_y_offset} ${Shank_z_offset}"/>
+            </xacro:unless>
+                <geometry>
+                    <cylinder length="${Shank_length}" radius="${Shank_radius}"/>
+                </geometry>
             </collision> -->
+            <collision>
+                <origin rpy="0 0 0" xyz="0 0 -0.033"/>
+                <geometry>
+                    <box size="${foot_width} ${foot_length} ${foot_height}"/>
+                </geometry>
+            </collision>
             <inertial>
                 <origin rpy="0 0 0" xyz="0.0 0.0 -0.01"/>

File: src/legged_examples/legged_unitree/legged_unitree_description/urdf/robot.urdf (robot description, URDF)
Before this commit: robot robot, 18 links, 17 joints
Links:
- link L_Foot: geometry collision box size=0.16 0.042 0.016; visual mesh filename=package://legged_unitree_description/meshes/a1/L_foot_drawi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 scale=1 1 1
- link R_Foot: geometry collision box size=0.16 0.042 0.016; visual mesh filename=package://legged_unitree_description/meshes/a1/R_foot_drawi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 scale=1 1 1

Commit message: gazebo is ok

File: src/legged_examples/legged_unitree/legged_unitree_description/urdf/a1/const.xacro (robot description, xacro)
@@ -44,5 +44,5 @@
     <xacro:property name="Thigh_z_offset" value="-0.17"/>
     <xacro:property name="Thigh_ry_offset" value="0"/>
-    <xacro:property name="foot_width" value="0.16"/>
+    <xacro:property name="foot_width" value="0.3"/>
     <xacro:property name="foot_length" value="0.042"/>
     <xacro:property name="foot_height" value="0.016"/>

File: src/legged_examples/legged_unitree/legged_unitree_description/urdf/robot.urdf (robot description, URDF)
Before this commit: robot robot, 18 links, 17 joints
Links:
- link L_Foot: geometry collision box size=0.3 0.042 0.016; visual mesh filename=package://legged_unitree_description/meshes/a1/L_foot_drawi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 scale=1 1 1
- link R_Foot: geometry collision box size=0.3 0.042 0.016; visual mesh filename=package://legged_unitree_description/meshes/a1/R_foot_drawi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 scale=1 1 1
Joints:
- joint L_JAnkle: limit lower=-3 upper=3 effort=33.5 velocity=33.5 -> lower=-3 upper=3 effort=33.5 velocity=21
- joint L_JHipRx: limit lower=-3 upper=3 effort=33.5 velocity=33.5 -> lower=-3 upper=3 effort=33.5 velocity=21
- joint L_JKnee: limit lower=-3 upper=3 effort=33.5 velocity=33.5 -> lower=-3 upper=3 effort=33.5 velocity=21
- joint L_JThigh: limit lower=-3 upper=3 effort=33.5 velocity=33.5 -> lower=-3 upper=3 effort=33.5 velocity=21
- joint R_JAnkle: limit lower=-3 upper=3 effort=33.5 velocity=33.5 -> lower=-3 upper=3 effort=33.5 velocity=21
- joint R_JHipRx: limit lower=-3 upper=3 effort=33.5 velocity=33.5 -> lower=-3 upper=3 effort=33.5 velocity=21
- joint R_JKnee: limit lower=-3 upper=3 effort=33.5 velocity=33.5 -> lower=-3 upper=3 effort=33.5 velocity=21
- joint R_JThigh: limit lower=-3 upper=3 effort=33.5 velocity=33.5 -> lower=-3 upper=3 effort=33.5 velocity=21
