Commit message: gazebo unsteady

File: src/legged_examples/legged_unitree/legged_unitree_description/urdf/a1/const.xacro (robot description, xacro)
@@ -44,7 +44,8 @@
     <xacro:property name="Thigh_z_offset" value="-0.17"/>
     <xacro:property name="Thigh_ry_offset" value="0"/>
-    <xacro:property name="foot_width" value="0.3"/>
-    <xacro:property name="foot_length" value="0.042"/>
+    <xacro:property name="foot_width" value="0.08"/>
+    <xacro:property name="foot_length" value="0.08"/>
     <xacro:property name="foot_height" value="0.016"/>
+    <xacro:property name="foot_x_offset" value="0.08"/>
     <!-- kinematic value -->
     <xacro:property name="thigh_offset" value="0.0838"/>
@@ -75,5 +76,5 @@
     <xacro:property name="trunk_mass" value="6.5"/>
     <xacro:property name="trunk_com_x" value="0.0000"/>
-    <xacro:property name="trunk_com_y" value="0.0"/>
+    <xacro:property name="trunk_com_y" value="0.017"/>
     <xacro:property name="trunk_com_z" value="0.15"/>
     <xacro:property name="trunk_ixx" value="0.3006167"/>

File: src/legged_examples/legged_unitree/legged_unitree_description/urdf/common/leg.xacro (robot description, xacro)
@@ -171,45 +171,33 @@
                 <material name="orange"/>
             </visual>
-            <!-- <visual>
-                <geometry>
-                    <sphere radius="0.001"/>
-                </geometry>
-                <origin xyz="0.125 0.0 -0.033" rpy="0 0 0"/>
-            </visual> -->
+            <collision>
+                <geometry>
+                    <sphere radius="0.02"/>
+                </geometry>
+                <origin xyz="-0.1 0.0 -0.03" rpy="0 0 0"/>
+            </collision>
+            <collision>
+                <geometry>
+                    <sphere radius="0.02"/>
+                </geometry>
+                <origin xyz="0.12 0.0 -0.03" rpy="0 0 0"/>
+            </collision>
             <!-- <collision>
-                <geometry>
-                    <sphere radius="0.02"/>
-                </geometry>
-                <origin xyz="0.01 0.0 -0.033" rpy="0 0 0"/>
+                <origin rpy="0 0 0" xyz="0 0 -0.033"/>
+                <geometry>
+                    <box size="${foot_width} ${foot_length} ${foot_height}"/>
+                </geometry>
+            </collision>             -->
+            <!-- <collision>
+            <xacro:if value="${(mirror == True)}">
+                <origin rpy="0 0 0" xyz="${foot_width} ${Shank_y_offset} ${Shank_z_offset}"/>
+            </xacro:if>
+            <xacro:unless value="${(mirror == False)}">
+                <origin rpy="0 0 0" xyz="${Shank_x_offset} ${-Shank_y_offset} ${Shank_z_offset}"/>
+            </xacro:unless>
+                <geometry>
+                    <cylinder length="${Shank_length}" radius="${Shank_radius}"/>
+                </geometry>
             </collision> -->
-            <!-- <visual>
-                <geometry>
-                    <sphere radius="0.001"/>
-                </geometry>
-                <origin xyz="-0.025 0.0 -0.033" rpy="0 0 0"/>
-            </visual>-->
-            <!-- <collision>
-                <geometry>
-                    <sphere radius="0.02"/>
-                </geometry>
-                <origin xyz="-0.01 0.0 -0.033" rpy="0 0 0"/>
-            </collision>  -->
-            <!-- <collision>
-            <xacro:if value="${(mirror == True)}">
-                <origin rpy="0 0 0" xyz="${foot_width} ${Shank_y_offset} ${Shank_z_offset}"/>
-            </xacro:if>
-            <xacro:unless value="${(mirror == False)}">
-                <origin rpy="0 0 0" xyz="${Shank_x_offset} ${-Shank_y_offset} ${Shank_z_offset}"/>
-            </xacro:unless>
-                <geometry>
-                    <cylinder length="${Shank_length}" radius="${Shank_radius}"/>
-                </geometry>
-            </collision> -->
-            <collision>
-                <origin rpy="0 0 0" xyz="0 0 -0.033"/>
-                <geometry>
-                    <box size="${foot_width} ${foot_length} ${foot_height}"/>
-                </geometry>
-            </collision>
             <inertial>
                 <origin rpy="0 0 0" xyz="0.0 0.0 -0.01"/>
@@ -250,6 +238,6 @@
         </gazebo>
         <gazebo reference="${prefix}_Foot">
-            <mu1>0.2</mu1>
-            <mu2>0.2</mu2>
+            <mu1>0.6</mu1>
+            <mu2>0.6</mu2>
             <material>Gazebo/DarkGrey</material>
             <kp value="1000000.0"/>

File: src/legged_examples/legged_unitree/legged_unitree_description/urdf/robot.urdf (robot description, URDF)
Before this commit: robot robot, 18 links, 17 joints
Links:
- link L_Foot: geometry collision sphere radius=0.02; collision sphere radius=0.02
- link R_Foot: geometry collision sphere radius=0.02; collision sphere radius=0.02
Joints:
- joint L_JHipRz: origin xyz=0 0.075 0 rpy=0 0 0 -> xyz=0 0.1 0 rpy=0 0 0
- joint R_JHipRz: origin xyz=0 -0.075 0 rpy=0 0 0 -> xyz=0 -0.1 0 rpy=0 0 0

File: src/legged_examples/legged_unitree/legged_unitree_description/urdf/robot.xacro (robot description, xacro)
@@ -32,8 +32,8 @@
     <xacro:IMU connected_to="base" imu_name="unitree_imu" xyz="0. 0. 0." rpy="0. 0. 0."/>
     <xacro:leg prefix="L" mirror="1" mirror_dae="False" front_hind="1" front_hind_dae="True">
-        <origin rpy="0 0 0" xyz="0 0.075 0"/>
+        <origin rpy="0 0 0" xyz="0 0.1 0"/>
     </xacro:leg>
     <xacro:leg prefix="R" mirror="-1" mirror_dae="True" front_hind="1" front_hind_dae="True">
-        <origin rpy="0 0 0" xyz="0 -0.075 0"/>
+        <origin rpy="0 0 0" xyz="0 -0.1 0"/>
     </xacro:leg>
     <xacro:arm prefix="L" mirror="1.0" mirror_dae="False" front_hind="1" front_hind_dae="True">

Commit message: all origin is set 0

File: src/legged_examples/legged_unitree/legged_unitree_description/urdf/a1/const.xacro (robot description, xacro)
@@ -76,5 +76,5 @@
     <xacro:property name="trunk_mass" value="6.5"/>
     <xacro:property name="trunk_com_x" value="0.0000"/>
-    <xacro:property name="trunk_com_y" value="0.017"/>
+    <xacro:property name="trunk_com_y" value="0.0"/>
     <xacro:property name="trunk_com_z" value="0.15"/>
     <xacro:property name="trunk_ixx" value="0.3006167"/>

File: src/legged_examples/legged_unitree/legged_unitree_description/urdf/common/arm.xacro (robot description, xacro)
@@ -37,5 +37,5 @@
             </collision>
             <inertial>
-                <origin rpy="0 0 0" xyz="0.01 0.0 0.0"/>
+                <origin rpy="0 0 0" xyz="0.0 0.0 0.0"/>
                 <mass value="0.30"/>
                 <inertia

File: src/legged_examples/legged_unitree/legged_unitree_description/urdf/common/leg.xacro (robot description, xacro)
@@ -145,5 +145,5 @@
             </collision>
             <inertial>
-                <origin rpy="0 0 0" xyz="-0.03416 -0.00075 -0.01"/>
+                <origin rpy="0 0 0" xyz="-0.0 -0.0 -0.01"/>
                 <mass value="0.70"/>
                 <inertia

Commit message: gazebo correct

File: src/legged_examples/legged_unitree/legged_unitree_description/urdf/a1/const.xacro (robot description, xacro)
@@ -44,5 +44,5 @@
     <xacro:property name="Thigh_z_offset" value="-0.17"/>
     <xacro:property name="Thigh_ry_offset" value="0"/>
-    <xacro:property name="foot_width" value="0.08"/>
+    <xacro:property name="foot_width" value="0.22"/>
     <xacro:property name="foot_length" value="0.08"/>
     <xacro:property name="foot_height" value="0.016"/>

File: src/legged_examples/legged_unitree/legged_unitree_description/urdf/common/arm.xacro (robot description, xacro)
@@ -151,5 +151,5 @@
             <kd value="100.0"/>
         </gazebo>
-        <gazebo reference="${prefix}_LShoulderRx">
+        <gazebo reference="${prefix}_LUpperArm">
             <mu1>0.2</mu1>
             <mu2>0.2</mu2>
@@ -158,5 +158,5 @@
             <kd value="100.0"/>
         </gazebo>
-        <gazebo reference="${prefix}_LUpperArm">
+        <gazebo reference="${prefix}_LForeArm">
             <mu1>0.2</mu1>
             <mu2>0.2</mu2>

File: src/legged_examples/legged_unitree/legged_unitree_description/urdf/common/leg.xacro (robot description, xacro)
@@ -171,5 +171,5 @@
                 <material name="orange"/>
             </visual>
-            <collision>
+            <!-- <collision>
                 <geometry>
                     <sphere radius="0.02"/>
@@ -182,11 +182,11 @@
                 </geometry>
                 <origin xyz="0.12 0.0 -0.03" rpy="0 0 0"/>
-            </collision>
-            <!-- <collision>
+            </collision>  -->
+            <collision>
                 <origin rpy="0 0 0" xyz="0 0 -0.033"/>
                 <geometry>
                     <box size="${foot_width} ${foot_length} ${foot_height}"/>
                 </geometry>
-            </collision>             -->
+            </collision>
             <!-- <collision>
             <xacro:if value="${(mirror == True)}">

File: src/legged_examples/legged_unitree/legged_unitree_description/urdf/robot.urdf (robot description, URDF)
Before this commit: robot robot, 18 links, 17 joints
Links:
- link L_Foot: geometry collision box size=0.22 0.08 0.016; visual mesh filename=package://legged_unitree_description/meshes/a1/L_foot_drawi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 scale=1 1 1
- link R_Foot: geometry collision box size=0.22 0.08 0.016; visual mesh filename=package://legged_unitree_description/meshes/a1/R_foot_drawi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 scale=1 1 1

Commit message: today happy

File: src/legged_examples/legged_unitree/legged_unitree_description/urdf/a1/const.xacro (robot description, xacro)
@@ -76,5 +76,5 @@
     <xacro:property name="trunk_mass" value="6.5"/>
     <xacro:property name="trunk_com_x" value="0.0000"/>
-    <xacro:property name="trunk_com_y" value="0.017"/>
+    <xacro:property name="trunk_com_y" value="0.0"/>
     <xacro:property name="trunk_com_z" value="0.15"/>
     <xacro:property name="trunk_ixx" value="0.3006167"/>

File: src/legged_examples/legged_unitree/legged_unitree_description/urdf/robot.urdf (robot description, URDF)
Before this commit: robot robot, 18 links, 17 joints
Joints:
- joint L_JAnkle: limit lower=-3 upper=3 effort=33.5 velocity=21 -> lower=-3 upper=3 effort=33.5 velocity=3
- joint L_JForeArm: limit lower=-3 upper=3 effort=33.5 velocity=33.5 -> lower=-3 upper=3 effort=33.5 velocity=21
- joint L_JUpperArm: limit lower=-3 upper=3 effort=33.5 velocity=33.5 -> lower=-3 upper=3 effort=33.5 velocity=21
- joint R_JAnkle: limit lower=-3 upper=3 effort=33.5 velocity=21 -> lower=-3 upper=3 effort=33.5 velocity=3
- joint R_JForeArm: limit lower=-3 upper=3 effort=33.5 velocity=33.5 -> lower=-3 upper=3 effort=33.5 velocity=21
- joint R_JUpperArm: limit lower=-3 upper=3 effort=33.5 velocity=33.5 -> lower=-3 upper=3 effort=33.5 velocity=21

Commit message: KalmanFilterEstimate::update: a_ b_ q_ are wrong

File: src/legged_examples/legged_unitree/legged_unitree_description/urdf/a1/const.xacro (robot description, xacro)
@@ -32,4 +32,10 @@
     <xacro:property name="HipRx_z_offset" value="-0.0"/>
     <xacro:property name="HipRx_ry_offset" value="1.57"/>
+    <xacro:property name="HipRz_radius" value="0.04"/>
+    <xacro:property name="HipRz_length" value="0.05"/>
+    <xacro:property name="HipRz_x_offset" value="0"/>
+    <xacro:property name="HipRz_y_offset" value="0"/>
+    <xacro:property name="HipRz_z_offset" value="0"/>
+    <xacro:property name="HipRz_ry_offset" value="1.57"/>
     <xacro:property name="Shank_radius" value="0.04"/>
     <xacro:property name="Shank_length" value="0.2"/>

File: src/legged_examples/legged_unitree/legged_unitree_description/urdf/common/leg.xacro (robot description, xacro)
@@ -28,4 +28,15 @@
                         izz="0.01355"/>
             </inertial>
+            <collision>
+            <xacro:if value="${(mirror == True)}">
+                <origin rpy="0 ${HipRz_ry_offset} 0" xyz="${HipRz_x_offset} ${HipRz_y_offset} ${HipRz_z_offset}"/>
+            </xacro:if>
+            <xacro:unless value="${(mirror == False)}">
+                <origin rpy="0 ${HipRz_ry_offset} 0" xyz="${HipRz_x_offset} ${HipRz_y_offset} ${HipRz_z_offset}"/>
+            </xacro:unless>
+                <geometry>
+                    <cylinder length="${HipRz_length}" radius="${HipRz_radius}"/>
+                </geometry>
+            </collision>
         </link>
         <joint name="${prefix}_JHipRx" type="revolute">

File: src/legged_examples/legged_unitree/legged_unitree_description/urdf/robot.urdf (robot description, URDF)
Before this commit: robot robot, 18 links, 17 joints
Links:
- link L_LHipRz: geometry collision cylinder length=0.05 radius=0.04; visual mesh filename=package://legged_unitree_description/meshes/a1/L_HipRz.obj scale=1 1 1
- link R_LHipRz: geometry collision cylinder length=0.05 radius=0.04; visual mesh filename=package://legged_unitree_description/meshes/a1/R_HipRz.obj scale=1 1 1

Commit message: command line

File: src/legged_examples/legged_unitree/legged_unitree_description/urdf/a1/const.xacro (robot description, xacro)
@@ -32,12 +32,12 @@
     <xacro:property name="HipRx_z_offset" value="-0.0"/>
     <xacro:property name="HipRx_ry_offset" value="1.57"/>
-    <xacro:property name="HipRz_radius" value="0.04"/>
+    <xacro:property name="HipRz_radius" value="0.02"/>
     <xacro:property name="HipRz_length" value="0.05"/>
     <xacro:property name="HipRz_x_offset" value="0"/>
     <xacro:property name="HipRz_y_offset" value="0"/>
-    <xacro:property name="HipRz_z_offset" value="0"/>
+    <xacro:property name="HipRz_z_offset" value="-0.1"/>
     <xacro:property name="HipRz_ry_offset" value="1.57"/>
     <xacro:property name="Shank_radius" value="0.04"/>
-    <xacro:property name="Shank_length" value="0.2"/>
+    <xacro:property name="Shank_length" value="0.15"/>
     <xacro:property name="Shank_x_offset" value="-0.0"/>
     <xacro:property name="Shank_y_offset" value="-0.0"/>

File: src/legged_examples/legged_unitree/legged_unitree_description/urdf/robot.urdf (robot description, URDF)
Before this commit: robot robot, 18 links, 17 joints
Links:
- link L_Foot: geometry collision box size=0.22 0.04 0.016; visual mesh filename=package://legged_unitree_description/meshes/a1/L_foot_drawi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 scale=1 1 1
- link L_LHipRz: geometry collision cylinder length=0.05 radius=0.02; visual mesh filename=package://legged_unitree_description/meshes/a1/L_HipRz.obj scale=1 1 1
- link L_LShank: geometry collision cylinder length=0.15 radius=0.04; visual mesh filename=package://legged_unitree_description/meshes/a1/L_LowerLeg3_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 scale=1 1 1
- link R_Foot: geometry collision box size=0.22 0.04 0.016; visual mesh filename=package://legged_unitree_description/meshes/a1/R_foot_drawi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 scale=1 1 1
- link R_LHipRz: geometry collision cylinder length=0.05 radius=0.02; visual mesh filename=package://legged_unitree_description/meshes/a1/R_HipRz.obj scale=1 1 1
- link R_LShank: geometry collision cylinder length=0.15 radius=0.04; visual mesh filename=package://legged_unitree_description/meshes/a1/R_LowerLeg3_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 scale=1 1 1

Commit message: 炸了

File: src/legged_examples/legged_unitree/legged_unitree_description/urdf/a1/const.xacro (robot description, xacro)
@@ -3,4 +3,5 @@
     <!-- Constants for robot dimensions -->
     <xacro:property name="stick_mass" value="0.00001"/>
+<xacro:property name="foot_radius" value="0.02"/>
     <!-- <xacro:property name="trunk_width" value="0.08"/>
     <xacro:property name="trunk_length" value="0.22"/>

File: src/legged_examples/legged_unitree/legged_unitree_description/urdf/common/leg.xacro (robot description, xacro)
@@ -184,16 +184,16 @@
             <!--  两个点 -->
             <!---->
-            <collision>
-                <geometry>
-                    <sphere radius="0.02"/>
-                </geometry>
-                <origin xyz="-0.1 0.0 -0.03" rpy="0 0 0"/>
-            </collision>
-            <collision>
-                <geometry>
-                    <sphere radius="0.02"/>
-                </geometry>
-                <origin xyz="0.12 0.0 -0.03" rpy="0 0 0"/>
-            </collision>
+<!--            <collision>-->
+<!--                <geometry>-->
+<!--                    <sphere radius="0.02"/>-->
+<!--                </geometry>-->
+<!--                <origin xyz="-0.1 0.0 -0.03" rpy="0 0 0"/>-->
+<!--            </collision>-->
+<!--            <collision>-->
+<!--                <geometry>-->
+<!--                    <sphere radius="0.02"/>-->
+<!--                </geometry>-->
+<!--                <origin xyz="0.12 0.0 -0.03" rpy="0 0 0"/>-->
+<!--            </collision>-->
             <!--  条形 -->
 <!--            <collision>-->
@@ -223,4 +223,64 @@
             </inertial>
         </link>
+        <joint name="${prefix}F_Jfoot_fixed" type="fixed">
+            <origin rpy="0 0 0" xyz="0.12 0.0 -0.03"/>
+            <parent link="${prefix}_Foot"/>
+            <child link="${prefix}F_Lfoot_fixed"/>
+        </joint>
+        <link name="${prefix}F_Lfoot_fixed">
+            <visual>
+                <origin rpy="0 0 0" xyz="0 0 0"/>
+                <geometry>
+                    <sphere radius="${0.01}"/>
+                </geometry>
+                <material name="orange"/>
+            </visual>
+            <collision>
+                <origin rpy="0 0 0" xyz="0 0 0"/>
+                <geometry>
+                    <sphere radius="${0.02}"/>
+                </geometry>
+            </collision>
+            <inertial>
+                <mass value="${foot_mass}"/>
+                <inertia
+                        ixx="${(2*foot_mass)/5.0*(foot_radius*foot_radius)}" ixy="0.0" ixz="0.0"
+                        iyy="${(2*foot_mass)/5.0*(foot_radius*foot_radius)}" iyz="0.0"
+                        izz="${(2*foot_mass)/5.0*(foot_radius*foot_radius)}"/>
+            </inertial>
+        </link>
+        <joint name="${prefix}H_Jfoot_fixed" type="fixed">
+            <origin rpy="0 0 0" xyz="-0.1 0.0 -0.03"/>
+            <parent link="${prefix}_Foot"/>
+            <child link="${prefix}H_Lfoot_fixed"/>
+        </joint>
+        <link name="${prefix}H_Lfoot_fixed">
+            <visual>
+                <origin rpy="0 0 0" xyz="0 0 0"/>
+                <geometry>
+                    <sphere radius="${0.01}"/>
+                </geometry>
+                <material name="orange"/>
+            </visual>
+            <collision>
+                <origin rpy="0 0 0" xyz="0 0 0"/>
+                <geometry>
+                    <sphere radius="${0.02}"/>
+                </geometry>
+            </collision>
+            <inertial>
+                <mass value="${foot_mass}"/>
+                <inertia
+                        ixx="${(2*foot_mass)/5.0*(foot_radius*foot_radius)}" ixy="0.0" ixz="0.0"
+                        iyy="${(2*foot_mass)/5.0*(foot_radius*foot_radius)}" iyz="0.0"
+                        izz="${(2*foot_mass)/5.0*(foot_radius*foot_radius)}"/>
+            </inertial>
+        </link>
+        <gazebo reference="${prefix}F_Lfoot_fixed">
+            <disableFixedJointLumping>true</disableFixedJointLumping>
+        </gazebo>
+        <gazebo reference="${prefix}H_Lfoot_fixed">
+            <disableFixedJointLumping>true</disableFixedJointLumping>
+        </gazebo>
         <gazebo reference="${prefix}_LHipRz">
             <mu1>0.2</mu1>

File: src/legged_examples/legged_unitree/legged_unitree_description/urdf/robot.urdf (robot description, URDF)
Before this commit: robot robot, 18 links, 17 joints
Links:
- added link LF_Lfoot_fixed; collision sphere radius=0.02; visual sphere radius=0.01
- added link LH_Lfoot_fixed; collision sphere radius=0.02; visual sphere radius=0.01
- added link RF_Lfoot_fixed; collision sphere radius=0.02; visual sphere radius=0.01
- added link RH_Lfoot_fixed; collision sphere radius=0.02; visual sphere radius=0.01
- link L_Foot: geometry visual mesh filename=package://legged_unitree_description/meshes/a1/L_foot_drawi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 scale=1 1 1
- link R_Foot: geometry visual mesh filename=package://legged_unitree_description/meshes/a1/R_foot_drawi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 scale=1 1 1
Joints:
- added joint LF_Jfoot_fixed: type fixed, parent L_Foot, child LF_Lfoot_fixed, origin xyz=0.12 0.0 -0.03 rpy=0 0 0
- added joint LH_Jfoot_fixed: type fixed, parent L_Foot, child LH_Lfoot_fixed, origin xyz=-0.1 0.0 -0.03 rpy=0 0 0
- added joint RF_Jfoot_fixed: type fixed, parent R_Foot, child RF_Lfoot_fixed, origin xyz=0.12 0.0 -0.03 rpy=0 0 0
- added joint RH_Jfoot_fixed: type fixed, parent R_Foot, child RH_Lfoot_fixed, origin xyz=-0.1 0.0 -0.03 rpy=0 0 0
